File: Kicad_axolitiLaser/AxolotiLaser.sch (KiCad schematic (older format))
At the start: 23 parts, among them J1 AudioJack3_SwitchTR, J2 AudioJack3_SwitchTR, J3 AudioJack3_SwitchTR, U1 TL072, U2 TL072, U3 TL072

Commit message: minor fixes
Parts:
- added J?: Conn_01x15, symbol Connector_Generic:Conn_01x15
- added J? (x2): Conn_01x03, symbol Connector_Generic:Conn_01x03
- added J?: DB25_Male, symbol Connector:DB25_Male
Connections:
- net GND: now also J?.1 (Pin_1)
- net Ax_Ring_OUT: now reaches J1.R, U1.5 (+)
- net Ax_Ring_OUT: now also J?.3 (Pin_3)
- net Ax_Tip_OUT: now reaches J1.T, U1.3 (+)
- net Ax_Tip_OUT: now also J?.2 (Pin_2); no longer R1.2
- net at RV1.1, U1.2 (-): now also R1.2
Other:
- moved on the sheet: J1, J2, J3, J?, R1, R11, R12, R13, R14, R15, R16, R17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
